File: KiCad/Line follower.kicad_pcb (KiCad board)
At the start: 2 copper layers, 80 x 90.5 mm, 67 parts, among them J1 USB_C_Receptacle_USB2.0_16P, J4 B2B-XH-A, U1 TCRT5000L, U10 TCRT5000L, U11 L298N, U2 ESP32-S3-WROOM-1, U3 TCRT5000L, U4 TCRT5000L, U5 TCRT5000L, U6 AMS1117-3.3, U7 TCRT5000L, U8 TCRT5000L, U9 TCRT5000L

Commit message: Dodanie brakujacych plikow
Parts:
- renumbered S1 to BOOT, H6 to IN, H9 to IN, H8 to OUT, H7 to OUT, J4 to POWER, S2 to RESET, S3 to START
Connections:
- U2 pad 10: unconnected-(U2-IO17-Pad10) -> /EnA
- U2 pad 11: unconnected-(U2-IO18-Pad11) -> /EnB
- U2 pad 32: /EnA -> unconnected-(U2-IO39-Pad32)
- U2 pad 33: /EnB -> unconnected-(U2-IO40-Pad33)
Routing:
- net /EnB: track 58.6 -> 79.9 mm
- net /EnA: track 56.9 -> 75.9 mm
- net /MOTORB IN: track 37.4 -> 40.2 mm
- net GND: track 113.5 -> 116.2 mm
- net /MOTORB OUT: track 51.0 -> 52.2 mm
- net /VCC_5V: track 186.3 -> 185.2 mm
Other:
- board text added: "BARTOSZ ZAWŁOCKI STEROWNIKI MIKROPROCESOROWE LINE FOLLOWER 2025/2026"
- board text added: "BÓG HONOR MECHATRONIKA"
